File: docs/aux_board/aux_board.kicad_sch (KiCad schematic)
At the start: 7 parts, among them J1 Conn_01x08_Pin, J2 Conn_01x05_Pin

Commit message: latence encoder
Connections:
- net 3.3V: now reaches J1.1 (Pin_1), R1.2, R2.2, U2.3 (LV)
- net Gnd: now reaches J1.2 (Pin_2), U1.2 (CA), U1.3 (E), U2.4 (GND), U3.2 (CA), U3.3 (E)
- net Gnd: now also J2.2 (Pin_2), U2.10 (GND)
- net CO1: now reaches J1.3 (Pin_3), U1.4 (CO)
- net CO2: now reaches J1.4 (Pin_4), U3.4 (CO)
- net Ch A: now reaches J1.5 (Pin_5), U2.1 (LV1)
- net Ch A: now also J2.5 (Pin_5), U2.7 (HV1)
- net Ch B: now reaches J1.6 (Pin_6), U2.2 (LV2)
- net Ch B: now also J2.4 (Pin_4), U2.8 (HV2)
- net Ch I: now reaches J1.7 (Pin_7), U2.5 (LV3)
- net Ch I: now also J2.1 (Pin_1), U2.11 (HV3)
- net 5V: now reaches J1.8 (Pin_8), J2.3 (Pin_3), U2.9 (HV)
Changed lines of the file:
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@@
+		)
+	)
+	(label "CO2"
+		(at 144.78 40.64 270)
+		(effects
+			(font
+				(size 1.27 1.27)
+			)
+			(justify right bottom)
+		)
+	)
+	(label "Ch B"
+		(at 81.28 87.63 0)
+		(effects
+			(font
+				(size 1.27 1.27)
+			)
+			(justify left bottom)
+		)
+	)
+	(label "Ch B"
+		(at 139.7 40.64 270)
+		(effects
+			(font
+				(size 1.27 1.27)
+			)
+			(justify right bottom)
+		)
+	)
+	(label "Ch I"
+		(at 137.16 40.64 270)
+		(effects
+			(font
+				(size 1.27 1.27)
+			)
+			(justify right bottom)
+		)
+	)
+	(label "3.3V"
+		(at 152.4 40.64 270)
+		(effects
+			(font
+				(size 1.27 1.27)
+			)
+			(justify right bottom)
+		)
+	)
+	(label "CO1"
+		(at 147.32 40.64 270)
+		(effects
+			(font
+				(size 1.27 1.27)
+			)
+			(justify right bottom)
+		)
+	)
+	(label "Ch A"
+		(at 81.28 90.17 0)
+		(effects
+			(font
+				(size 1.27 1.27)
+			)
+			(justify left bottom)
+		)
+	)
+	(label "5V"
+		(at 134.62 40.64 270)
+		(effects
+			(font
+				(size 1.27 1.27)
+			)
+			(justify right bottom)
+		)
+	)
+	(label "Vcc"
+		(at 81.28 85.09 0)
+		(effects
+			(font
+				(size 1.27 1.27)
+			)
+			(justify left bottom)
+		)
+	)
+	(label "Ch A"
+		(at 142.24 40.64 270)
+		(effects
+			(font
+				(size 1.27 1.27)
+			)
+			(justify right bottom)
+		)
+	)
+	(label "Ch I"
+		(at 81.28 80.01 0)
+		(effects
+			(font
+				(size 1.27 1.27)
+			)
+			(justify left bottom)
+		)
+	)
+	(label "Gnd"
+		(at 149.86 40.64 270)
+		(effects
+			(font
+				(size 1.27 1.27)
+			)
+			(justify right bottom)
+		)
+	)
+	(label "Gnd"
+		(at 81.28 82.55 0)
+		(effects
+			(font
+				(size 1.27 1.27)
+			)
+			(justify left bottom)
 		)
 	)

Commit message: webapp error
Parts:
- removed U2: (no value), symbol optek:LevelShifter
- added C1: 18pF, symbol Device:C_Small_US
- added C2: 18 pF, symbol Device:C_Small_US
- added R3: 1M, symbol Device:R
- added U3: LS7366R-S, LS7366R-S:SOIC127P600X175-14N, symbol LS7366R-S:LS7366R-S
- added Y1: 40 MHz, symbol Device:Crystal
- renumbered U3 to U2
Connections:
- net CO2: no longer J1.4 (Pin_4)
- net 3.3V renamed +3V3
- net 5V renamed +5V
- net +5V: now also U3.14 (VDD)
- net Ch A: no longer names the net of J1.5 (Pin_5)
- net Ch A: no longer J2.5 (Pin_5)
- net Ch B: no longer names the net of J1.6 (Pin_6)
- net Ch B: no longer J2.4 (Pin_4)
- net Ch I: no longer names the net of J1.7 (Pin_7)
- net Ch I: no longer J2.1 (Pin_1)
- net Gnd renamed GND
- net GND: now also C1.2, C2.2, U3.3 (VSS)
- new net: C1.1, R3.2, Y1.1
- new net: C2.1, R3.1, Y1.2
- new net CH A: J2.5 (Pin_5)
- new net CH B: J2.4 (Pin_4)
- new net CH I: J2.1 (Pin_1)
Other:
- note added: "Capteurs fin course"
- note added: "Vers GPIO RPi"
- note added: "Vers Moteur"
- moved on the sheet: J1, J2, R1, R2, U1, U2

Commit message: pcb
Parts:
- removed J1: Conn_01x08_Pin, symbol Connector:Conn_01x08_Pin
- added C3: 0.1uF, symbol Device:C_Small_US
- added J1: SPI et GPIO interfaces, Connector_PinHeader_2.54mm:PinHeader_2x05_P2.54mm_Vertical, symbol Connector_Generic:Conn_02x05_Odd_Even
- added JP1, JP2: Jumper_2_Bridged, symbol Jumper:Jumper_2_Bridged
- added R4, R5: 1K, symbol Device:R
- J2: value Conn_01x05_Pin -> Encoder Interface; footprint (none) -> Connector_PinHeader_2.54mm:PinHeader_1x05_P2.54mm_Vertical
- R1, R2: value R -> 220
- U3: footprint LS7366R-S:SOIC127P600X175-14N -> Package_SO:SOIC-14_3.9x8.7mm_P1.27mm
- Y1: footprint (none) -> Crystal:Crystal_SMD_2520-4Pin_2.5x2.0mm
Connections:
- net CH A is gone; now on net A_1: J2.5 (Pin_5)
- net CH B is gone; now on net B_1: J2.4 (Pin_4)
- net CH I is gone; now on net I_1: J2.1 (Pin_1)
- net +3V3: now also J1.8 (Pin_8)
- net +5V: now also C3.1, J1.10 (Pin_10), JP1.1 (A), JP2.1 (A)
- net CO1: now also J1.2 (Pin_2)
- net CO2: now also J1.4 (Pin_4)
- net GND: now also C3.2, J1.9 (Pin_9)
- net FSCKO_1: now reaches C1.1, R3.2, Y1.1
- net FSCKO_1: now also U3.1 (FCKO)
- net FSCKI_1: now reaches C2.1, R3.1, Y1.2
- net FSCKI_1: now also U3.2 (FCKI)
- net I_1: now reaches U3.10 (INDEX/)
- net B_1: now reaches U3.11 (B)
- net B_1: now also R5.2
- net A_1: now reaches U3.12 (A)
- net A_1: now also R4.2
- net CNT_EN_1: now reaches U3.13 (CNT_EN)
- net CNT_EN_1: now also J1.6 (Pin_6)
- net S1: now reaches U3.4 (SS/)
- net S1: now also J1.1 (Pin_1)
- net SCLK: now reaches U3.5 (SCK)
- net SCLK: now also J1.7 (Pin_7)
- net MISO: now reaches U3.6 (MISO)
- net MISO: now also J1.5 (Pin_5)
- net MOSI: now reaches U3.7 (MOSI)
- net MOSI: now also J1.3 (Pin_3)
- net LFLAG_1: now reaches U3.8 (LFLAG/)
- net DFLAG_1: now reaches U3.9 (DFLAG/)
- new net: JP2.2 (B), R5.1
- new net: JP1.2 (B), R4.1
Other:
- note added: "Compteur tours"
- moved on the sheet: C1, C2, J2, R3, U3, Y1

Commit message: pcb
Parts:
- removed C3: 0.1uF, symbol Device:C_Small_US
- removed J1: SPI et GPIO interfaces, Connector_PinHeader_2.54mm:PinHeader_2x05_P2.54mm_Vertical, symbol Connector_Generic:Conn_02x05_Odd_Even
- removed JP1, JP2: Jumper_2_Bridged, symbol Jumper:Jumper_2_Bridged
- removed R4, R5: 1K, symbol Device:R
- added J1: Conn_01x08_Pin, symbol Connector:Conn_01x08_Pin
- J2: value Encoder Interface -> Conn_01x05_Pin; footprint Connector_PinHeader_2.54mm:PinHeader_1x05_P2.54mm_Vertical -> (none)
- R1, R2: value 220 -> R
- U3: footprint Package_SO:SOIC-14_3.9x8.7mm_P1.27mm -> LS7366R-S:SOIC127P600X175-14N
- Y1: footprint Crystal:Crystal_SMD_2520-4Pin_2.5x2.0mm -> (none)
Connections:
- net +3V3: now also J1.1 (Pin_1)
- net +5V: now also J1.8 (Pin_8)
- net CO1: now also J1.3 (Pin_3)
- net GND: now also J1.2 (Pin_2)
- net A_1: no longer names the net of U3.12 (A)
- net A_1: no longer J2.5 (Pin_5)
- net B_1: no longer names the net of U3.11 (B)
- net B_1: no longer J2.4 (Pin_4)
- net CNT_EN_1: no longer names the net of U3.13 (CNT_EN)
- net DFLAG_1: no longer names the net of U3.9 (DFLAG/)
- net FSCKI_1: no longer names the net of C2.1, R3.1, Y1.2
- net FSCKI_1: no longer U3.2 (FCKI)
- net FSCKO_1: no longer names the net of C1.1, R3.2, Y1.1
- net FSCKO_1: no longer U3.1 (FCKO)
- net I_1: no longer names the net of U3.10 (INDEX/)
- net I_1: no longer J2.1 (Pin_1)
- net LFLAG_1: no longer names the net of U3.8 (LFLAG/)
- net MISO: no longer names the net of U3.6 (MISO)
- net MOSI: no longer names the net of U3.7 (MOSI)
- net S1: no longer names the net of U3.4 (SS/)
- net SCLK: no longer names the net of U3.5 (SCK)
- new net CH A: J2.5 (Pin_5)
- new net CH B: J2.4 (Pin_4)
- new net CH I: J2.1 (Pin_1)
Other:
- note removed: "Compteur tours"
- moved on the sheet: C1, C2, J2, R3, U3, Y1
